File: Excelsior488nm_Controller_Schematic.brd (EAGLE design)
At the start: 87.6 x 85.1 mm, 14 parts

Commit message: Revision B
Parts:
- added R5: 470, rcl:R0603
- added R6, R7, R8: 1k, rcl:R0603
- R1, R2, R3: value 560 -> 1k
- R4: value 560 -> 670
- moved JP1 19.1 mm to (55.9, 39.4)
- moved JP2 19.1 mm to (55.9, 45.7)
- moved JP3 19.1 mm to (55.9, 53.3)
- moved IC 19.1 mm to (35.6, 49.5)
- moved ALARM 19.0 mm to (90.2, 54.6)
- moved EMISSION 19.0 mm to (90.2, 73.7)
- moved LASER_ON 19.0 mm to (90.2, 10.2)
- moved OUTPUT_OK 19.0 mm to (90.2, 33.0)
- moved R1 19.0 mm to (69.8, 43.2)
- moved R2 19.0 mm to (69.8, 48.3)
- moved R3 19.0 mm to (69.8, 72.4)
- moved R4 19.0 mm to (69.8, 53.3)
- moved S1 19.0 mm to (64.8, 22.9)
Connections:
- removed net N$13: IC.9, SV1.4
- new net N$4: IC.9, R8.1, SV1.4
- net +5V: now also R5.2, R6.2, R7.2, R8.2
- net N$2: now also R6.1
- net N$3: now also R7.1
- net N$9: now also R5.1
Routing:
- net N$1: track 54.2 -> 37.3 mm
- net +5V: track 21.6 -> 37.3 mm
- net N$13: track 9.63 -> 0.00 mm
- net GND: track 230.7 -> 237.0 mm
Other:
- board size 87.6 x 85.1 mm -> 111.8 x 85.1 mm

Commit message: Schematic update
Parts:
- removed IC: 7414D, 74xx-us:SO14
- added IC1, IC2, IC3: 74LVC1G04DCK, 74xx-little-de:SC70-5
- added PIN14: (no value), pinhead:1X01
- R5: value 470 -> 1k
- R8: value 1k -> 470
- SV1: device con-lstb:MA04-1 -> con-lstb:MA03-1
- moved SV1 57.2 mm to (6.35, -8.89), turned to 0 degrees
- renumbered JP1 to PIN2, JP2 to PIN1, JP3 to PIN10
Connections:
- removed net N$4: IC.9, R8.1, SV1.4
- new net PIN2: IC3.2, PIN2.1, R5.1, S1.2
- net +5V: now also IC1.5, IC2.5, IC3.5; no longer IC.11, IC.13, IC.14
- net GND: now also IC1.3, IC2.3, IC3.3; no longer IC.5, IC.7
- net N$1: now also IC1.4; no longer IC.8
- net N$2: now also IC1.2, PIN14.1, R7.1; no longer IC.1, PIN2.1, R6.1, S1.2
- net N$3: now also IC2.2, R6.1; no longer IC.3, R7.1
- net N$7: now also IC3.4; no longer IC.2
- net N$8: now also IC2.4; no longer IC.4
- net N$9: now also R8.1; no longer R5.1
Routing:
- net GND: track 237.0 -> 178.9 mm
- net N$2: track 42.3 -> 0.00 mm
- net +5V: track 37.3 -> 0.00 mm
- net N$1: track 37.3 -> 0.00 mm
- net N$8: track 30.9 -> 3.49 mm
- net PIN2: track 0.00 -> 18.8 mm
- net N$3: track 18.3 -> 0.00 mm
- net N$9: track 13.1 -> 0.00 mm
- net N$7: track 31.9 -> 24.9 mm

Commit message: Board layout
Parts:
- ALARM, EMISSION, LASER_ON, OUTPUT_OK: device led:LED10MM -> led:LED3MM
- moved IC1 93.8 mm to (79.2, 41.8), turned to 270 degrees
- moved R8 86.0 mm to (104.1, 41.9), turned to 90 degrees
- moved PIN14 81.4 mm to (69.8, 41.9)
- moved IC2 78.8 mm to (52.1, 41.9), turned to 270 degrees
- moved IC3 71.5 mm to (24.1, 41.9), turned to 270 degrees
- moved LASER_ON 64.3 mm to (34.3, 41.9)
- moved SV1 48.3 mm to (3.81, 39.4), turned to 90 degrees
- moved R5 47.0 mm to (19.1, 41.9), turned to 90 degrees
- moved PIN10 43.4 mm to (97.8, 41.9)
- moved R1 41.9 mm to (27.9, 41.9), turned to 90 degrees
- moved R4 41.0 mm to (109.2, 41.9), turned to 90 degrees
- moved PIN2 40.7 mm to (15.2, 41.9)
- moved R7 37.0 mm to (74.9, 41.9), turned to 90 degrees
- moved R3 33.5 mm to (83.8, 41.9), turned to 90 degrees
- moved EMISSION 31.8 mm to (90.2, 41.9)
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Routing:
- net +5V: track 0.00 -> 135.8 mm
- net N$6: track 43.8 -> 5.43 mm
- net N$12: track 32.7 -> 5.43 mm
- net PIN2: track 18.8 -> 41.6 mm
- net N$7: track 24.9 -> 3.04 mm
- net N$11: track 18.7 -> 5.43 mm
- net N$9: track 0.00 -> 11.8 mm
- net N$10: track 18.7 -> 7.97 mm
- net GND: track 178.9 -> 188.6 mm
- net N$2: track 0.00 -> 9.30 mm
- net N$3: track 0.00 -> 8.74 mm
- net N$1: track 0.00 -> 3.75 mm
Other:
- board size 111.8 x 85.1 mm -> 125.7 x 49.5 mm
