File: Excelsior488nm_Controller_Schematic.sch (EAGLE design)
At the start: 11 parts

Commit message: Finalized 488-1A
Parts:
- removed J1: (no value), con-jack:DCJ0303
- removed X1: (no value), con-subd:F15HDV
- added JP1, JP2, JP3: (no value), pinhead:PINHD-1X1
- added S1: (no value), switch:M9040P
- added SV1: (no value), con-lstb:MA04-1
Connections:
- removed net N$4: ICC.I, X1.14
- removed net N$5: ICA.O, R1.1
- new net N$13: ICC.I, SV1.4
- new net N$8: ICE.O, R2.1
- net +5V: now also ICA.I, ICB.I, SV1.3; no longer J1.1
- net GND: now also S1.S, SV1.1, SV1.2; no longer ICD.I, ICE.I, J1.3, X1.6
- net N$2: now also ICD.I, JP1.1, S1.P; no longer ICA.I, X1.2
- net N$3: now also ICE.I, JP2.1; no longer ICB.I, X1.1
- net N$7: now also ICD.O, R1.1; no longer ICB.O, R2.1
- net N$9: now also JP3.1; no longer X1.10
Other:
- note added: "488-1"
- note added: "A"
- note added: "DESIGN NOTES"
- note added: "ICA-ICF: SN74HC14 6-CH INVERTER"
- note added: "LEDS: RED, V_f=1.8V, I_f = 10mA MAX"
- note added: "Laser GND"
- note added: "Laser PIN 1"
- note added: "Laser PIN 10"
- note added: "Laser PIN 14"
- note added: "Laser PIN 2"
- note added: "PS +5VDC"
- note added: "PS GND"
- note added: "Tyler Camp"
- moved on the sheet: ALARM, EMISSION, ICA, ICB, ICC, ICD, ICE, ICF, ICP, LASER_ON, OUTPUT_OK, R1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

Commit message: Revision B
Parts:
- added R5: 470, rcl:R-US_R0603
- added R6, R7, R8: 1k, rcl:R-US_R0603
- R1, R2, R3: value 560 -> 1k
- R4: value 560 -> 670
Connections:
- removed net N$13: ICC.I, SV1.4
- new net N$4: ICC.I, R8.1, SV1.4
- net +5V: now also R5.2, R6.2, R7.2, R8.2
- net N$2: now also R6.1
- net N$3: now also R7.1
- net N$9: now also R5.1
Other:
- note added: "B"
- note removed: "A"
- moved on the sheet: ALARM, EMISSION, ICA, ICB, ICC, ICD, ICE, ICF, ICP, JP1, JP2, JP3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

Commit message: Schematic update
Parts:
- removed IC: 7414D, 74xx-us:7414D
- removed JP3: (no value), pinhead:PINHD-1X1
- added IC1, IC2, IC3: 74LVC1G04DCK, 74xx-little-de:74LVC1G04DCK
- added PIN10, PIN14: (no value), pinhead:PINHD-1X1
- R5: value 470 -> 1k
- R8: value 1k -> 470
- SV1: device con-lstb:MA04-1 -> con-lstb:MA03-1
- renumbered JP1 to PIN2, JP2 to PIN1
Connections:
- removed net N$4: ICC.I, R8.1, SV1.4
- new net PIN2: IC3A.I, PIN2.1, R5.1, S1.P
- net +5V: now also IC1P.VCC, IC2P.VCC, IC3P.VCC; no longer ICA.I, ICB.I, ICP.VCC
- net GND: now also IC1P.GND, IC2P.GND, IC3P.GND; no longer ICF.I, ICP.GND
- net N$1: now also IC1A.O; no longer ICC.O
- net N$2: now also IC1A.I, PIN14.1, R7.1; no longer ICD.I, PIN2.1, R6.1, S1.P
- net N$3: now also IC2A.I, R6.1; no longer ICE.I, R7.1
- net N$7: now also IC3A.O; no longer ICD.O
- net N$8: now also IC2A.O; no longer ICE.O
- net N$9: now also PIN10.1, R8.1; no longer JP3.1, R5.1
Other:
- note removed: "Laser PIN 1"
- note removed: "Laser PIN 10"
- note removed: "Laser PIN 14"
- note removed: "Laser PIN 2"
- moved on the sheet: R5, R6, R7, R8

Commit message: Board layout
Parts:
- ALARM, EMISSION, LASER_ON, OUTPUT_OK: device led:LED10MM -> led:LED3MM
Changed lines of the file:
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@@
 <part name="R3" library="rcl" library_urn="urn:adsk.eagle:library:334" deviceset="R-US_" device="R0603" package3d_urn="urn:adsk.eagle:package:23555/3" value="1k"/>
 <part name="R4" library="rcl" library_urn="urn:adsk.eagle:library:334" deviceset="R-US_" device="R0603" package3d_urn="urn:adsk.eagle:package:23555/3" value="670"/>
-<part name="LASER_ON" library="led" library_urn="urn:adsk.eagle:library:259" deviceset="LED" device="10MM" package3d_urn="urn:adsk.eagle:package:15828/1"/>
-<part name="OUTPUT_OK" library="led" library_urn="urn:adsk.eagle:library:259" deviceset="LED" device="10MM" package3d_urn="urn:adsk.eagle:package:15828/1"/>
-<part name="EMISSION" library="led" library_urn="urn:adsk.eagle:library:259" deviceset="LED" device="10MM" package3d_urn="urn:adsk.eagle:package:15828/1"/>
-<part name="ALARM" library="led" library_urn="urn:adsk.eagle:library:259" deviceset="LED" device="10MM" package3d_urn="urn:adsk.eagle:package:15828/1"/>
+<part name="LASER_ON" library="led" library_urn="urn:adsk.eagle:library:259" deviceset="LED" device="3MM" package3d_urn="urn:adsk.eagle:package:15797/1"/>
+<part name="OUTPUT_OK" library="led" library_urn="urn:adsk.eagle:library:259" deviceset="LED" device="3MM" package3d_urn="urn:adsk.eagle:package:15797/1"/>
+<part name="EMISSION" library="led" library_urn="urn:adsk.eagle:library:259" deviceset="LED" device="3MM" package3d_urn="urn:adsk.eagle:package:15797/1"/>
+<part name="ALARM" library="led" library_urn="urn:adsk.eagle:library:259" deviceset="LED" device="3MM" package3d_urn="urn:adsk.eagle:package:15797/1"/>
 <part name="PIN2" library="pinhead" library_urn="urn:adsk.eagle:library:325" deviceset="PINHD-1X1" device="" package3d_urn="urn:adsk.eagle:package:22485/2"/>
 <part name="PIN1" library="pinhead" library_urn="urn:adsk.eagle:library:325" deviceset="PINHD-1X1" device="" package3d_urn="urn:adsk.eagle:package:22485/2"/>
